File: james_ewing_ee_design_take_home/High_Side_Switch_and_Current_Measurement.kicad_sch (KiCad schematic)
At the start: 13 parts, among them Q1 PMOS, Q2 NMOS, U6 MAX4080F, U7 OPA320AQDBVRQ1

Commit message: Updated
Parts:
- removed R19: 2, symbol Device:R
- removed U7: OPA320AQDBVRQ1, Package_SON:Texas_S-PVSON-N10, symbol Amplifier_Audio:OPA1622
- added D3: STTH30L06G-TR, symbol Device:D
- R23: value 100k -> 1k
Connections:
- net GND: now also D3.2 (A)
- net Vfet: now also D3.1 (K)
- net at U6.5 (OUT): now also R17.2
- net at R21.1, R22.2: now also Q1.2 (G)
Other:
- note added: "ADC on ESP8266 is 10bit giving us a range of 0 to 1023. This results in a 9.765mA resolution."
- note added: "Flyback Diode chosen so its reverse polarity voltage rating is 10x the nominal voltage. The diode current rating is also 3x the nominal load current."
- note added: "OUT is low impedance since it's the output of an Op-AMP gain stage, so no additional Op-AMP needed to drive V_imeas."
- note added: "V_thresholdmax = -20V V_thresholdmin = -4V"
- note added: "Voltage Divider needed to prevent Vgs exceeding -20V, 15V chosen as safe max, and to max sure we exceed the miller plateau voltage for the FET of -4V. Min voltage therefore chosen to be -6V."
- note removed: "ADC on ESP8266 is 10bit giving us a range of 0 to 1023. This results in a 9.775mA resolution."
- note removed: "Op AMP Supply: V(+) 5V V(-) GND"
- note removed: "Op-AMP allows clean ADC sampling even at higher frequency as Op-AMP isolates R17, R18, and C14 from rest of circuit."
- note removed: "Voltage Divider needed to prevent Vgs exceeding 20V. Need to choose values that still puts Vgs lower bound at 4V or greater."
- title: (none) -> Local High Side Switch and Current Measurement Circuit
- moved on the sheet: C14, Q1, R17, R18

Commit message: Updated Schematic
Parts:
- added D4: 10V Zener, symbol Device:D_Zener
- Q1: value PMOS -> SQM100P10-19L_GE3
- R21: value 2M -> 10k
- R22: value 1M -> 100k
Connections:
- net Vfet: now also D4.1 (K); no longer D3.1 (K)
- net Vout: now also D3.1 (K)
- net at Q1.2 (G), R21.1, R22.2: now also D4.2 (A)
Other:
- note added: "TODO: Calculate Gate Capacitance and see if there will be issues with too slow charge/discharge."
- note added: "V_thresholdmax = -20V V_thresholdmin = -4V ( 4V ~ Miller Plateau)"
- note removed: "V_thresholdmax = -20V V_thresholdmin = -4V"
- note removed: "Voltage Divider needed to prevent Vgs exceeding -20V, 15V chosen as safe max, and to max sure we exceed the miller plateau voltage for the FET of -4V. Min voltage therefore chosen to be -6V."
- moved on the sheet: Q1
