File: james_ewing_ee_design_take_home/Local_RS485_Interface.kicad_sch (KiCad schematic)
At the start: 28 parts, among them J1 USB_B_Micro, J3 RJ45, J5 Conn_Coaxial, U1 ESP8266EX, U1 SN65176BDR, U5 M95M02-DR, Y2 TSX-3225

Commit message: Updated
Other:
- note added: "ADC on ESP8266 is 10bit giving us a range of 0 to 1023. This results in a 9.765mA resolution."
- note added: "ESP8266 Microcontroller"
- note added: "Terminating Resistor"
- note removed: "ADC on ESP8266 is 10bit giving us a range of 0 to 1023. This results in a 9.775mA resolution."
- title: (none) -> Local Interface Communication Circuit
Changed lines of the file:
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@@
 (kicad_sch (version 20230121) (generator eeschema)
   (paper "A4")
+  (title_block
+    (title "Local Interface Communication Circuit")
+  )
   (junction (at 100.33 95.25) (diameter 0) (color 0 0 0 0)
   )
@@
     (effects (font (size 1.27 1.27)) (justify left bottom))
   )
-  (text "ADC on ESP8266 is 10bit giving us \na range of 0 to 1023. This results\nin a 9.775mA resolution. "
+  (text "ADC on ESP8266 is 10bit giving us \na range of 0 to 1023. This results\nin a 9.765mA resolution. "
     (at 111.76 77.47 0)
     (effects (font (size 1.27 1.27)) (justify left bottom))
@@
   )
   (text "Chip Enable" (at 91.44 86.36 0)
+    (effects (font (size 1.27 1.27)) (justify left bottom))
+  )
+  (text "Terminating \nResistor" (at 64.77 168.91 0)
     (effects (font (size 1.27 1.27)) (justify left bottom))
   )
@@
     (effects (font (size 1.27 1.27)) (justify right bottom))
   )
+  (text "ESP8266 Microcontroller" (at 60.96 20.32 0)
+    (effects (font (size 2 2)) (justify right bottom))
+  )
   (text "Mysterious Circuit that \nturns 5V to 3.3V :)" (at 201.93 60.96 0)

Commit message: Updated Schematic
Parts:
- added C15: 1uF, symbol Device:C
- added C5: 0.22uF, symbol Device:C
- added C6: 10uF, symbol Device:C
- added R11, R19, R24, R25: 10k, symbol Device:R
- added R27, R28, R29: 0, symbol Device:R
- added SW1, SW2, SW3: RST, symbol Switch:SW_Push
- added U2: MCP2200-E-SS, Package_SO:SSOP-20_5.3x7.2mm_P0.65mm, symbol Interface_USB:MCP2200-E-SS
- added Y1: Resonator, symbol Device:Resonator
Connections:
- net 3v3: now also R19.1, R24.2
- net GND: now also C15.1, C5.2, C6.2, R25.2, SW1.2, SW2.2, SW3.2, U2.20 (VSS), Y1.2
- net TX_RX_SEL: now also R27.2
- net UART_RX: now also R28.1
- net UART_TX: now also R29.1
- net at U1.13 (MTDO): now also R25.1
- net GPI0: now reaches U1.15 (GPIO0)
- net GPI0: now also R24.1, SW3.1
- net LNA: now reaches C10.1, L2.1, U1.2 (LNA)
- net RST: now reaches U1.32 (~{EXT_RSTB})
- net RST: now also C15.2, R19.2, SW1.1
- net at R7.1, U1.7 (CHIP_PU): now also SW2.1
- net D_Minus: now reaches J1.2 (D-)
- net D_Minus: now also U2.18 (D-)
- net D_Plus: now reaches J1.3 (D+)
- net D_Plus: now also U2.19 (D+)
- net 5V renamed 5V_LI
- net 5V_LI: now also C6.1, R11.2, U2.1 (VDD)
- new net: R11.1, U2.4 (RST)
- new net: C5.1, U2.17 (V_USB)
- new net: U2.2 (OSC1), Y1.3
- new net: U2.3 (OSC2), Y1.1
- new net TX_RX_SEL_PROG: R27.1, U2.14 (GP2)
- new net UART_RX_PROG: R29.2, U2.12 (RX)
- new net UART_TX_PROG: R28.2, U2.10 (TX)
- no-connect marks 19 -> 23
Other:
- note added: "12MHz Resonator for USB"
- note added: "BOOT"
- note added: "C16 Bypass CAP needed since only powering off BUS Voltage."
- note added: "DON'T POPULATE SW1 (Unless Using RST for RESET)"
- note added: "Decided to not connect the LEDs."
- note added: "EN"
- note added: "GPIO15"
- note added: "Keep Trace as Short as Possible"
- note added: "Reccomended to RESET with EN"
- note added: "Resistors Removeable after Programming"
- note added: "TODO: Add 5V to 3.3V regulator."
- note added: "TODO: Add BLINK LED for Testing"
- note added: "USB to UART Interface for Programming"
- note removed: "Chip Enable"
- moved on the sheet: C1, C2, C7, C8, D1, J3, L1, R1, R12, R2, R3, R4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
