File: james_ewing_ee_design_take_home/High_Side_Switch_and_Current_Measurement_GateDriver.kicad_sch (KiCad schematic)
At the start: 19 parts, among them J6 TJ0251830000G, J7 TJ0251830000G, Q3 NMOS, U6 MAX4080F, U8 FAN7371

Commit message: Updated Documentation
Other:
- note added: "Version 2"
Changed lines of the file:
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@@
   )
   (text "High Side Switch" (at 21.59 74.93 0)
-    (effects (font (size 2 2)) (justify left bottom))
+    (effects (font (size 2 2) (thickness 0.4) bold) (justify left bottom))
   )
   (text "PWM Signal" (at 15.24 111.76 0)
@@
   )
   (text "Current Measurement" (at 20.32 29.21 0)
-    (effects (font (size 2 2)) (justify left bottom))
+    (effects (font (size 2 2) (thickness 0.4) bold) (justify left bottom))
   )
   (text "MAX Vgs = 20V\nDriver operates\nat 15V, allows \nRdson to be <\n8.2mOhm for very\nefficient operation."
@@
     (effects (font (size 1.27 1.27)) (justify left bottom))
   )
+  (text "Version 2" (at 177.8 171.45 0)
+    (effects (font (size 2.5 2.5) (thickness 0.5) bold) (justify left bottom))
+  )
   (text "E-NMOS" (at 99.06 113.03 0)
