File: james_ewing_ee_design_take_home/Power.kicad_sch (KiCad schematic)
At the start: 25 parts, among them U10 NCP59748MN1ADJTBG, U9 MP2492DN-LF-Z

Commit message: Updated Documentation
Other:
- note added: "28V to 15V Supply"
- note added: "28V to 5V Supply"
- note added: "5V to 3.3V Supply"
Changed lines of the file:
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@@
     (effects (font (size 0.75 0.75)) (justify left bottom))
+  )
+  (text "28V to 15V Supply" (at 38.1 91.44 0)
+    (effects (font (size 2 2) (thickness 0.4) bold) (justify left bottom))
   )
   (text "10nF sets soft start to 18ms, with open 0.2ms soft start."
@@
     (effects (font (size 1.27 1.27)) (justify left bottom))
   )
+  (text "5V to 3.3V Supply" (at 170.18 26.67 0)
+    (effects (font (size 2 2) (thickness 0.4) bold) (justify left bottom))
+  )
+  (text "28V to 5V Supply" (at 27.94 30.48 0)
+    (effects (font (size 2 2) (thickness 0.4) bold) (justify left bottom))
+  )
   (global_label "15V" (shape input) (at 63.5 102.87 0) (fields_autoplaced)
