File: james_ewing_ee_design_take_home/Remote_RS485_Interface.kicad_sch.kicad_sch (KiCad schematic)
At the start: 23 parts, among them J1 USB_B_Micro, J3 RJ45, U2 MCP2200-E-SS, U3 SN65176BDR, Y1 Resonator

Commit message: Updated Documentation
Changed lines of the file:
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@@
     (effects (font (size 1.27 1.27)) (justify left bottom))
   )
-  (text "USB to UART Interface" (at 36.83 27.94 0)
-    (effects (font (size 2 2)) (justify left bottom))
+  (text "USB to UART Interface" (at 35.56 30.48 0)
+    (effects (font (size 2 2) (thickness 0.4) bold) (justify left bottom))
   )
   (text "Transient Protection rated\nfor 1kV with TVS" (at 106.68 128.27 0)
@@
   )
   (text "UART to RS485 Interface" (at 34.29 115.57 0)
-    (effects (font (size 2 2)) (justify left bottom))
+    (effects (font (size 2 2) (thickness 0.4) bold) (justify left bottom))
   )
   (text "Twisted Pair chosen is \"Orange White\" and \"Orange\" \nwhich are Pin 1 and Pin 2 respectively. T568B Pinout Used."
@@
     (effects (font (size 1.27 1.27)) (justify left bottom))
   )
-  (text "12MHz Resonator for USB" (at 45.72 41.91 0)
+  (text "12MHz Resonator for USB" (at 46.99 41.91 0)
     (effects (font (size 1.27 1.27)) (justify left bottom))
   )
