File: james_ewing_ee_design_take_home_koenigsegg/Local_RS485_Interface.kicad_sch (KiCad schematic)
At the start: 45 parts, among them J1 USB_B_Micro, J3 RJ45, J5 Conn_Coaxial, SW1 RST, SW2 RST, SW3 RST, U1 ESP8266EX, U1 SN65176BDR, U2 MCP2200-E-SS, U5 M95M02-DR, Y1 Resonator, Y2 TSX-3225

Commit message: Implemented new Version
Parts:
- added D12, D3: Green LED 20mA, symbol Device:LED
- added R20, R21: 165, symbol Device:R
Connections:
- net GND: now also D12.1 (K), D3.1 (K)
- net TX_LED: now reaches U2.5 (GP7/TxLED)
- net TX_LED: now also R20.1
- net RX_LED: now reaches U2.6 (GP6/RxLED)
- net RX_LED: now also R21.1
- net BLINK_LED renamed EN_BUCK
- new net: D3.2 (A), R20.2
- new net: D12.2 (A), R21.2
- no-connect marks 22 -> 20
Other:
- note removed: "Decided to not connect the LEDs."
- note removed: "TEST LED"
- moved on the sheet: C1, C10, C11, C12, C13, C15, C2, C7, C8, C9, D1, D6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
