File: james_ewing_ee_design_take_home_koenigsegg/Remote_RS485_Interface.kicad_sch.kicad_sch (KiCad schematic)
At the start: 23 parts, among them J1 USB_B_Micro, J3 RJ45, U2 MCP2200-E-SS, U3 SN65176BDR, Y1 Resonator

Commit message: Implemented new Version
Other:
- note added: "James Ewing EE Design Challenge Remote Current Sense and High Side Switch"
- moved on the sheet: C1, C2, C36, C37, C5, C6, D1, D11, D6, J1, J3, R1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
