File: james_ewing_ee_design_take_home_koenigsegg/james_ewing_ee_design_take_home_koenigsegg.kicad_sch (KiCad schematic)
At the start: 0 parts

Commit message: Implemented new Version
Other:
- removed sheet High_Side_Switch_and_Current_Measurement_Zener
Changed lines of the file:
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@@
     (title "Remote Interface ")
   )
-  (sheet (at 342.9 474.98) (size 321.31 182.88) (fields_autoplaced)
+  (sheet (at 0 466.09) (size 321.31 182.88) (fields_autoplaced)
     (stroke (width 0.1524) (type solid))
     (fill (color 0 0 0 0.0000))
-    (property "Sheetname" "Power" (at 342.9 474.2684 0)
+    (property "Sheetname" "Power" (at 0 465.3784 0)
       (effects (font (size 1.27 1.27)) (justify left bottom))
     )
-    (property "Sheetfile" "Power.kicad_sch" (at 342.9 658.4446 0)
+    (property "Sheetfile" "Power.kicad_sch" (at 0 649.5546 0)
       (effects (font (size 1.27 1.27)) (justify left top))
     )
     (instances
-      (project "james_ewing_ee_design_take_home"
-        (path "/bb8655b5-ca3d-4aaf-8979-cdbfbb70a000" (page "6"))
+      (project "james_ewing_ee_design_take_home_koenigsegg"
+        (path "/bb8655b5-ca3d-4aaf-8979-cdbfbb70a000" (page "5"))
       )
     )
   )
-  (sheet (at 344.17 238.76) (size 318.77 194.31) (fields_autoplaced)
+  (sheet (at 342.9 245.11) (size 316.23 184.15) (fields_autoplaced)
     (stroke (width 0.1524) (type solid))
     (fill (color 0 0 0 0.0000))
-    (property "Sheetname" "High_Side_Switch_and_Current_Measurement_Zener" (at 344.17 238.0484 0)
+    (property "Sheetname" "High_Side_Switch_and_Current_Measurement_GateDriver" (at 342.9 244.3984 0)
       (effects (font (size 1.27 1.27)) (justify left bottom))
     )
-    (property "Sheetfile" "High_Side_Switch_and_Current_Measurement_Zener.kicad_sch" (at 344.17 433.6546 0)
+    (property "Sheetfile" "High_Side_Switch_and_Current_Measurement_GateDriver.kicad_sch" (at 342.9 429.8446 0)
       (effects (font (size 1.27 1.27)) (justify left top))
     )
     (instances
-      (project "james_ewing_ee_design_take_home"
+      (project "james_ewing_ee_design_take_home_koenigsegg"
         (path "/bb8655b5-ca3d-4aaf-8979-cdbfbb70a000" (page "4"))
-      )
-    )
-  )
-  (sheet (at 2.54 476.25) (size 297.18 184.15) (fields_autoplaced)
-    (stroke (width 0.1524) (type solid))
-    (fill (color 0 0 0 0.0000))
-    (property "Sheetname" "High_Side_Switch_and_Current_Measurement_GateDriver" (at 2.54 475.5384 0)
-      (effects (font (size 1.27 1.27)) (justify left bottom))
-    )
-    (property "Sheetfile" "High_Side_Switch_and_Current_Measurement_GateDriver.kicad_sch" (at 2.54 660.9846 0)
-      (effects (font (size 1.27 1.27)) (justify left top))
-    )
-    (instances
-      (project "james_ewing_ee_design_take_home"
-        (path "/bb8655b5-ca3d-4aaf-8979-cdbfbb70a000" (page "5"))
       )
     )
@@
     )
     (instances
-      (project "james_ewing_ee_design_take_home"
+      (project "james_ewing_ee_design_take_home_koenigsegg"
         (path "/bb8655b5-ca3d-4aaf-8979-cdbfbb70a000" (page "2"))
       )
     )
   )
-  (sheet (at 2.54 238.76) (size 295.91 193.04) (fields_autoplaced)
+  (sheet (at 2.54 238.76) (size 314.96 193.04) (fields_autoplaced)
     (stroke (width 0.1524) (type solid))
     (fill (color 0 0 0 0.0000))
@@
     )
     (instances
-      (project "james_ewing_ee_design_take_home"
+      (project "james_ewing_ee_design_take_home_koenigsegg"
         (path "/bb8655b5-ca3d-4aaf-8979-cdbfbb70a000" (page "3"))
       )
